File: face_plate/mxr_face_plate.kicad_pcb (KiCad board)
At the start: 2 copper layers, 20 x 128.5 mm, 10 parts

Commit message: JLC mark
Other:
- board text added: "JLCJLCJLCJLC"
Changed lines of the file:
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@@
   (gr_line (start 42.5 150) (end 53 150) (layer "F.SilkS") (width 0.3))
   (gr_line (start 53 142) (end 42.5 142) (layer "F.SilkS") (width 0.3))
+  (gr_text "JLCJLCJLCJLC" (at 50 43.5) (layer "B.SilkS")
+    (effects (font (size 1 1) (thickness 0.15)) (justify mirror))
+  )
   (zone (net 1) (net_name "GND") (layer "F.Cu") (hatch edge 0.508)
     (connect_pads yes (clearance 0))
