File: face_plate/mxr_face_plate.kicad_sch (KiCad schematic)
At the start: 10 parts

Commit message: faceplate
Parts:
- H101, H102, H103, H104: footprint WITNS:PotentiometerHole_7.4mm_M7_Pad_Via -> WITNS:PotentiometerHole_7.4mm_M7_Pad
- H105, H106, H107, H108, H109: footprint WITNS:Thonkiconn_6.4mm_M6_Pad_Via -> WITNS:Thonkiconn_6.4mm_M6_Pad
Changed lines of the file:
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@@
       (effects (font (size 1.27 1.27)) (justify left))
     )
-    (property "Footprint" "WITNS:Thonkiconn_6.4mm_M6_Pad_Via" (id 2) (at 113.03 85.09 0)
+    (property "Footprint" "WITNS:Thonkiconn_6.4mm_M6_Pad" (id 2) (at 113.03 85.09 0)
       (effects (font (size 1.27 1.27)) hide)
     )
@@
       (effects (font (size 1.27 1.27)) (justify left))
     )
-    (property "Footprint" "WITNS:PotentiometerHole_7.4mm_M7_Pad_Via" (id 2) (at 96.52 60.96 0)
+    (property "Footprint" "WITNS:PotentiometerHole_7.4mm_M7_Pad" (id 2) (at 96.52 60.96 0)
       (effects (font (size 1.27 1.27)) hide)
     )
@@
       (effects (font (size 1.27 1.27)) (justify left))
     )
-    (property "Footprint" "WITNS:Thonkiconn_6.4mm_M6_Pad_Via" (id 2) (at 104.14 85.09 0)
+    (property "Footprint" "WITNS:Thonkiconn_6.4mm_M6_Pad" (id 2) (at 104.14 85.09 0)
       (effects (font (size 1.27 1.27)) hide)
     )
@@
       (effects (font (size 1.27 1.27)) (justify left))
     )
-    (property "Footprint" "WITNS:PotentiometerHole_7.4mm_M7_Pad_Via" (id 2) (at 127 60.96 0)
+    (property "Footprint" "WITNS:PotentiometerHole_7.4mm_M7_Pad" (id 2) (at 127 60.96 0)
       (effects (font (size 1.27 1.27)) hide)
     )
@@
       (effects (font (size 1.27 1.27)) (justify left))
     )
-    (property "Footprint" "WITNS:Thonkiconn_6.4mm_M6_Pad_Via" (id 2) (at 96.52 85.09 0)
+    (property "Footprint" "WITNS:Thonkiconn_6.4mm_M6_Pad" (id 2) (at 96.52 85.09 0)
       (effects (font (size 1.27 1.27)) hide)
     )
@@
       (effects (font (size 1.27 1.27)) (justify left))
     )
-    (property "Footprint" "WITNS:PotentiometerHole_7.4mm_M7_Pad_Via" (id 2) (at 106.68 60.96 0)
+    (property "Footprint" "WITNS:PotentiometerHole_7.4mm_M7_Pad" (id 2) (at 106.68 60.96 0)
       (effects (font (size 1.27 1.27)) hide)
     )
@@
       (effects (font (size 1.27 1.27)) (justify left))
     )
-    (property "Footprint" "WITNS:Thonkiconn_6.4mm_M6_Pad_Via" (id 2) (at 121.92 85.09 0)
+    (property "Footprint" "WITNS:Thonkiconn_6.4mm_M6_Pad" (id 2) (at 121.92 85.09 0)
       (effects (font (size 1.27 1.27)) hide)
     )
@@
       (effects (font (size 1.27 1.27)) (justify left))
     )
-    (property "Footprint" "WITNS:PotentiometerHole_7.4mm_M7_Pad_Via" (id 2) (at 116.84 60.96 0)
+    (property "Footprint" "WITNS:PotentiometerHole_7.4mm_M7_Pad" (id 2) (at 116.84 60.96 0)
       (effects (font (size 1.27 1.27)) hide)
     )
@@
       (effects (font (size 1.27 1.27)) (justify left))
     )
-    (property "Footprint" "WITNS:Thonkiconn_6.4mm_M6_Pad_Via" (id 2) (at 129.54 85.09 0)
+    (property "Footprint" "WITNS:Thonkiconn_6.4mm_M6_Pad" (id 2) (at 129.54 85.09 0)
       (effects (font (size 1.27 1.27)) hide)
     )
@@
     )
     (path "/7402790f-0651-4f24-b9b3-e659446a7e5c"
-      (reference "H101") (unit 1) (value "CH1") (footprint "WITNS:PotentiometerHole_7.4mm_M7_Pad_Via")
+      (reference "H101") (unit 1) (value "CH1") (footprint "WITNS:PotentiometerHole_7.4mm_M7_Pad")
     )
     (path "/91dd6056-429c-4721-8430-2711727e5689"
-      (reference "H102") (unit 1) (value "CH2") (footprint "WITNS:PotentiometerHole_7.4mm_M7_Pad_Via")
+      (reference "H102") (unit 1) (value "CH2") (footprint "WITNS:PotentiometerHole_7.4mm_M7_Pad")
     )
     (path "/d1163dc3-bb72-4e39-9b2d-50117dd5bfe7"
-      (reference "H103") (unit 1) (value "CH3") (footprint "WITNS:PotentiometerHole_7.4mm_M7_Pad_Via")
+      (reference "H103") (unit 1) (value "CH3") (footprint "WITNS:PotentiometerHole_7.4mm_M7_Pad")
     )
     (path "/85df24db-26b9-47e8-a427-67f6f3fd9ba8"
-      (reference "H104") (unit 1) (value "CH4") (footprint "WITNS:PotentiometerHole_7.4mm_M7_Pad_Via")
+      (reference "H104") (unit 1) (value "CH4") (footprint "WITNS:PotentiometerHole_7.4mm_M7_Pad")
     )
     (path "/8af8243f-06fc-419e-a7bc-b42262a26e62"
-      (reference "H105") (unit 1) (value "I1") (footprint "WITNS:Thonkiconn_6.4mm_M6_Pad_Via")
+      (reference "H105") (unit 1) (value "I1") (footprint "WITNS:Thonkiconn_6.4mm_M6_Pad")
     )
     (path "/84d92d25-004a-4618-af96-0ece38fb5ec1"
-      (reference "H106") (unit 1) (value "I2") (footprint "WITNS:Thonkiconn_6.4mm_M6_Pad_Via")
+      (reference "H106") (unit 1) (value "I2") (footprint "WITNS:Thonkiconn_6.4mm_M6_Pad")
     )
     (path "/3d961422-1272-42c0-ac3e-a85cf6295001"
-      (reference "H107") (unit 1) (value "I3") (footprint "WITNS:Thonkiconn_6.4mm_M6_Pad_Via")
+      (reference "H107") (unit 1) (value "I3") (footprint "WITNS:Thonkiconn_6.4mm_M6_Pad")
     )
     (path "/c0abc96d-ed67-42c5-b30d-758bd90bed72"
-      (reference "H108") (unit 1) (value "I4") (footprint "WITNS:Thonkiconn_6.4mm_M6_Pad_Via")
+      (reference "H108") (unit 1) (value "I4") (footprint "WITNS:Thonkiconn_6.4mm_M6_Pad")
     )
     (path "/e15e5ba7-c922-4b5a-a676-a369e5deb577"
-      (reference "H109") (unit 1) (value "OUT") (footprint "WITNS:Thonkiconn_6.4mm_M6_Pad_Via")
-    )
-  )
+      (reference "H109") (unit 1) (value "OUT") (footprint "WITNS:Thonkiconn_6.4mm_M6_Pad")
+    )
+  )
